Commit message: fixed tf errors and updated robot model; additional script files in /scripts folder

File: robots/youbot.urdf.xacro (robot description, xacro)
@@ -23,34 +23,43 @@
   <xacro:include filename="$(find sick_tim)/urdf/sick_tim.urdf.xacro" />
   <xacro:include filename="$(find youbot_description)/urdf/sensors/asus_xtion_camera.urdf.xacro" />
-  <!-- Now we can start using the macros xacro:included above to define the actual youbot -->
-  <!-- The first use of a macro.  This one was defined in base.urdf.xacro above.
-       A macro like this will expand to a set of link and joint definitions, and to additional
-       Gazebo-related extensions (sensor plugins, etc).  The macro takes an argument, name,
-       that equals "base", and uses it to generate names for its component links and joints
-       (e.g., base_link).  The xacro:included origin block is also an argument to the macro.  By convention,
-       the origin block defines where the component is w.r.t its parent (in this case the parent
-       is the world frame). For more, see http://www.ros.org/wiki/xacro -->
-  <!-- foot for arm-->
-  <xacro:youbot_base name="base"/>
-  <xacro:youbot_plate name="plate" parent="base_link">
+  <!-- properties -->
+  <property name="base_name" value="base"/>
+  <property name="arm_name" value="arm"/>
+  <property name="laser_name" value="laser"/>
+  <property name="camera_name" value="camera"/>
+  <!-- youbot base link and joint-->
+  <link name="youbot_link" />
+  <joint name="youbot_base_joint" type="fixed">
+      <parent link="youbot_link" />
+      <child link="${base_name}_footprint" />
+  </joint>
+  <!-- youbot base files -->
+  <xacro:youbot_base name="${base_name}"/>
+  <xacro:youbot_plate name="plate" parent="${base_name}_link">
     <origin xyz="-0.159 0 0.046" rpy="0 0 0" />
   </xacro:youbot_plate>
-  <xacro:youbot_arm name="arm" parent="base_link">
+  <xacro:youbot_arm name="${arm_name}" parent="${base_name}_link">
     <origin xyz="0.143 0 0.046" rpy="0 0 0" />
   </xacro:youbot_arm>
-  <xacro:youbot_gripper name="gripper" parent="arm_link_5">
+  <xacro:youbot_gripper name="gripper" parent="${arm_name}_link_5">
     <origin xyz="0 0 0" rpy="0 0 0" />
   </xacro:youbot_gripper>
   <!-- camera at the gripper -->
-  <xacro:asus_xtion_camera name="camera" parent="arm_link_5" tilt="0" >
+  <xacro:asus_xtion_camera name="${camera_name}" parent="${arm_name}_link_5" tilt="0" >
     <!-- <origin xyz="-0.035 0 0.015" rpy="0 -1.57 0" /> -->
     <origin xyz="-0.035 0 0.005" rpy="0 -1.57 0" />
   </xacro:asus_xtion_camera>
+  <link name="camera_link" />
+  <joint name="camera_link_joint" type="fixed">
+      <origin xyz="0 0 0" rpy="0 0 0"/>
+      <parent link="${camera_name}_tilt_link" />
+      <child link="camera_link" />
+  </joint>
   <!-- base laser front -->
   <joint name="tim_mount_joint" type="fixed">
-      <parent link="base_link" />
-      <child link="laser_mount_link" />
+      <parent link="${base_name}_link" />
+      <child link="${laser_name}_mount_link" />
       <origin xyz="${0.04+base_size_x/2.0} 0 0.01" rpy="3.14 0 0"/>
   </joint>
-  <xacro:sick_tim551 name="laser" ros_topic="scan" />
+  <xacro:sick_tim551 name="${laser_name}" ros_topic="scan" />
 </robot>
